File: pcb/paperClockPCB.sch (KiCad schematic (older format))
At the start: 13 parts, among them J1 USB_B_Micro, J2 Conn_01x02_Female, J3 Conn_01x08, J4 Conn_01x02, J5 Conn_01x02, J6 AVR-ISP-6, M1 DS1337, U1 ATmega328P-PU, Y1 Crystal

Commit message: PCB v0.1
Connections:
- net GND: now also J1.6 (Shield)
- no-connect marks 14 -> 13
Changed lines of the file:
@@
 NoConn ~ 2050 2000
 NoConn ~ 2050 2100
-NoConn ~ 1650 2300
+$Comp
+L power:GND #PWR?
+U 1 1 5D787D3C
+P 1650 2400
+F 0 "#PWR?" H 1650 2150 50  0001 C CNN
+F 1 "GND" H 1655 2227 50  0000 C CNN
+F 2 "" H 1650 2400 50  0001 C CNN
+F 3 "" H 1650 2400 50  0001 C CNN
+	1    1650 2400
+	1    0    0    -1
+$EndComp
+Wire Wire Line
+	1650 2300 1650 2400
 $EndSCHEMATC
