File: pcb/paperClockPCB.kicad_pcb (KiCad board)
At the start: 2 copper layers, 13 parts, among them J1 USB_B_Micro, J2 Conn_01x02_Female, J3 Conn_01x08, J4 Conn_01x02, J5 Conn_01x02, J6 AVR-ISP-6, M1 DS1337, U1 ATmega328P-PU, Y1 Crystal

Commit message: PCB v0.1
Parts:
- added REF**: MountingHole_2.2mm_M2_ISO7380, MountingHole:MountingHole_2.2mm_M2_ISO7380, F.Cu at (136.4, 84.3)
- added REF**: MountingHole_2.2mm_M2_ISO7380, MountingHole:MountingHole_2.2mm_M2_ISO7380, F.Cu at (136.4, 52.3)
- moved J4 1.02 mm to (160.8, 52.6)
- moved J1 1.02 mm to (136.1, 76.2)
- moved C3 0.25 mm to (146.6, 68.8)
- moved C4 0.25 mm to (144.5, 51.6)
- moved J2 0.25 mm to (136.4, 61.2)
- moved J5 0.25 mm to (136.7, 67.3)
Connections:
- J1 pad 6: Net-(J1-Pad6) -> GND
Routing:
- net Net-(J6-Pad5): track 0.00 -> 32.3 mm, vias 0 -> 3
- net VCC: track 72.1 -> 69.9 mm
- net /TX: track 16.6 -> 15.9 mm
Other:
- board outline added: 29 x 36.6 mm

Commit message: PCB v0.1
Other:
- board text added: "JDM"
Changed lines of the file:
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@@
   (general
     (thickness 1.6)
-    (drawings 4)
+    (drawings 5)
     (tracks 120)
     (zones 0)
@@
   )
   (setup
-    (last_trace_width 0.508)
+    (last_trace_width 0.1524)
     (user_trace_width 0.254)
     (user_trace_width 0.381)
@@
     (descr "Through hole straight socket strip, 1x08, 2.54mm pitch, single row (from Kicad 4.0.7), script generated")
     (tags "Through hole socket strip THT 1x08 2.54mm single row")
-    (fp_text reference J3 (at -1.016 2.77 90) (layer B.SilkS)
+    (fp_text reference J3 (at -1.016 2.286 90) (layer B.SilkS)
       (effects (font (size 1 1) (thickness 0.15)) (justify mirror))
     )
@@
     )
   )
+  (gr_text JDM (at 143.256 58.674 90) (layer B.SilkS)
+    (effects (font (size 1.5 1.5) (thickness 0.3)) (justify mirror))
+  )
   (gr_line (start 134.112 86.614) (end 134.112 50.038) (layer Edge.Cuts) (width 0.15))
